File: hardware/01-power-supply/v5/kicad/sam17-power-v5.kicad_pcb (KiCad board)
At the start: 4 copper layers, 200 x 150 mm, 215 parts, among them J1 Bornera 2P 5.0 mm, J10 PinHeader 1x04, J2 Molex KK-254 4P, J3 Bornera 4P 5.08 mm, J5 Faston 6.3x0.8 PCB, J6 Molex KK-254 2P, J7 Molex KK-254 4P, J8 PinHeader 1x04, J9 Molex KK-254 2P, Q2 CSD18534Q5A, Q3 MMBT3906, Q4 MMBT3906, Q5 MMBT3906, Q6 MMBT3906, Q7 CSD18534Q5A, SW1 Pulsador 6x6, U1 LT1963AEQ, U10 ADS1115IDGS, U11 TMP1075DGK, U12 INA226, U13 INA226, U14 INA226, U15 LM74502DDFR, U16 TPS26631PWPR, U17 MSP430FR2111IPW16, U18 TPS70933DBVR, U19 TPS26631PWPR, U2 LT3015EQ, U20 LM393B, U21 TL431BI, U22 TL431BI, U23 TL431BI, U24 TL431BI, U25 TL431BI, U4 LT3045EDD, U5 LT3045EDD, U6 LT3094EDD, U7 LT3094EDD, U8 INA226, U9 ISO1541

Commit message: fuente-v5: R36 a 3,74 kohm, el OVP de U19 deja sitio al sobreimpulso del THN
R36 pasa de 3,9 kohm a 3,74 kohm 0,1 % (Yageo RT0805BRD073K74L, C865467,
misma serie y huella). El OVP de U19 sube de 16,55 a 17,21 V nominal, con
banda de 16,83 a 17,59 V: el margen sobre el THN sano pasa de 0,18 a 0,82 V
en la envolvente de margen_budget.py, y el sobreimpulso tipico al soltar
carga (~0,19 V) cabe.

Con el borde alto por encima del pico de #334 (17,40 V), lo peor que ve U1
es un THN atascado justo debajo del OVP. check_absmax.py toma el mayor de
los dos en absmax.csv, en la guarda de D10 y en su canario; D10 sigue sin
conducir (17,59 V contra V_BR 17,8 V).

La spec v5 y la propuesta de piezas llevan la banda nueva y las cifras del
disparo rapido (3,32 A, 7,5 us). Placa regenerada con --desde-ruteo: mismo
ruteo, DRC en 0.
Parts:
- R36: value 3.9k 0.1% -> 3.74k 0.1%
